File: maple_r6/pwr.sch (KiCad schematic (older format))
At the start: 20 parts, among them IC1 BQ24010DRC, IC2 MCP1700T, IC3 MCP1700T

Commit message: R6v1 : Updated schematic and created PCB layout
Parts:
- D3: value Red -> CHRG
- D4: value Green -> DONE
- External1: value PWR_JACK -> EXT
- LIPO1: value CONN_2 -> 3.7V LiPo
- PWR1: value CONN_4X2 -> PWRSEL
