File: maple_r6/stm32.sch (KiCad schematic (older format))
At the start: 40 parts, among them J1-A1 CONN_8, J1-B1 CONN_8, J2 CONN_6, J3-A1 CONN_8, J3-B1 CONN_8, J4 CONN_6, M2 CONN_2, Q2 NPN, Q3 NPN

Commit message: R6v1 : Updated schematic and created PCB layout
Parts:
- D1: value Blue -> D13
- JTAG1: value CONN_4X2 -> JTAG
- RESET1: value BUT -> RESET
- renumbered R25 to R3, R24 to R7
Connections:
- net +5V: now also J4.3
- net GND: now also JTAG1.2; no longer JTAG1.7
- net JTAG-TCK: now also JTAG1.3; no longer JTAG1.6
- net JTAG-TDI: now also JTAG1.5; no longer JTAG1.4
- net JTAG-TDO: now also JTAG1.4; no longer JTAG1.5
- net JTAG-TMS: now also JTAG1.6; no longer JTAG1.3
- net JTAG-TRST: no longer J4.1, JTAG1.1
- net RST: now also J4.1, JTAG1.1
- net VAA: no longer J4.3
- net VCC: now also JTAG1.7; no longer JTAG1.2
